Commit message: Add timestamp field

File: robosense_description/urdf/RS-16.urdf.xacro (robot description, xacro)
@@ -125,5 +125,5 @@
     <xacro:property name="imu_name" value="${name}_imu"/>
     <xacro:property name="imu_topic" value="/${name}/imu"/>
-    <xacro:property name="imu_hz" value="100"/>
+    <xacro:property name="imu_hz" value="200"/>
     <joint name="${imu_name}_joint" type="fixed">
       <parent link="${name}"/>
